File: lets_split.kicad_pcb (KiCad board)
At the start: 2 copper layers, 112 x 79 mm, 60 parts, among them J1 3PIN, J2 6PIN, J3 3PIN, SW1 SW_PUSH, SW10 SW_PUSH, SW11 SW_PUSH, SW12 SW_PUSH, SW13 SW_PUSH, SW14 SW_PUSH, SW15 SW_PUSH, SW16 SW_PUSH, SW17 SW_PUSH, SW18 SW_PUSH, SW19 SW_PUSH, SW2 SW_PUSH, SW21 SW_PUSH, SW22 SW_PUSH, SW23 SW_PUSH, SW3 SW_PUSH, SW4 SW_PUSH, SW5 SW_PUSH, SW6 SW_PUSH, SW7 SW_PUSH, SW8 SW_PUSH, SW9 SW_PUSH, U2 HOLE, U3 HOLE, U4 HOLE, U5 HOLE

Commit message: add revision on PCB
Other:
- board text added: "Cherry MX version Rev. develop"
- board text added: "for Holtite socket"
Changed lines of the file:
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@@
     (links 160)
     (no_connects 0)
-    (area 36.538572 31.635 149.075001 114.7216)
+    (area 36.924999 32.924999 149.075001 112.075001)
     (thickness 1.6)
-    (drawings 29)
+    (drawings 31)
     (tracks 380)
     (zones 0)
@@
     (pad "" np_thru_hole circle (at -1.65 -0.7) (size 2.1 2.1) (drill 2.1) (layers *.Cu *.Mask))
   )
+  (gr_text "for Holtite socket" (at 78.867 71.374) (layer B.SilkS)
+    (effects (font (size 1 1.4) (thickness 0.2)) (justify mirror))
+  )
+  (gr_text "Cherry MX version\nRev. develop" (at 148.336 109.601) (layer B.SilkS)
+    (effects (font (size 1 1) (thickness 0.2)) (justify left mirror))
+  )
   (gr_text "LET'S SPLIT" (at 90.75 75.5) (layer B.SilkS)

Commit message: first release
Other:
- board text added: "Cherry MX version Rev. 1.0.0"
- board text removed: "Cherry MX version Rev. develop"
Changed lines of the file:
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@@
     (links 160)
     (no_connects 0)
-    (area 36.924999 32.924999 149.075001 112.075001)
+    (area 36.538572 31.635 149.075001 114.7216)
     (thickness 1.6)
     (drawings 31)
@@
     (effects (font (size 1 1.4) (thickness 0.2)) (justify mirror))
   )
-  (gr_text "Cherry MX version\nRev. develop" (at 148.336 109.601) (layer B.SilkS)
+  (gr_text "Cherry MX version\nRev. 1.0.0" (at 148.336 109.601) (layer B.SilkS)
     (effects (font (size 1 1) (thickness 0.2)) (justify left mirror))
   )

Commit message: development version
Other:
- board text added: "Cherry MX version Rev. devel"
- board text removed: "Cherry MX version Rev. 1.0.0"
Changed lines of the file:
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@@
     (effects (font (size 1 1.4) (thickness 0.2)) (justify mirror))
   )
-  (gr_text "Cherry MX version\nRev. 1.0.0" (at 148.336 109.601) (layer B.SilkS)
+  (gr_text "Cherry MX version\nRev. devel" (at 148.336 109.601) (layer B.SilkS)
     (effects (font (size 1 1) (thickness 0.2)) (justify left mirror))
   )
