File: lets_split.kicad_pcb (KiCad board)
At the start: 2 copper layers, 112 x 79 mm, 60 parts, among them J1 3PIN, J2 6PIN, J3 3PIN, SW1 SW_PUSH, SW10 SW_PUSH, SW11 SW_PUSH, SW12 SW_PUSH, SW13 SW_PUSH, SW14 SW_PUSH, SW15 SW_PUSH, SW16 SW_PUSH, SW17 SW_PUSH, SW18 SW_PUSH, SW19 SW_PUSH, SW2 SW_PUSH, SW21 SW_PUSH, SW22 SW_PUSH, SW23 SW_PUSH, SW3 SW_PUSH, SW4 SW_PUSH, SW5 SW_PUSH, SW6 SW_PUSH, SW7 SW_PUSH, SW8 SW_PUSH, SW9 SW_PUSH, U2 HOLE, U3 HOLE, U4 HOLE, U5 HOLE

Commit message: bump version to 1.0.1
Other:
- board text added: "Cherry MX version Rev. 1.0.1"
- board text removed: "Cherry MX version Rev. devel"
Changed lines of the file:
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@@
     (links 160)
     (no_connects 0)
-    (area 36.924999 32.924999 149.075001 112.075001)
+    (area 36.538572 31.635 149.075001 114.7216)
     (thickness 1.6)
     (drawings 31)
@@
     (effects (font (size 1 1.4) (thickness 0.2)) (justify mirror))
   )
-  (gr_text "Cherry MX version\nRev. devel" (at 148.336 109.601) (layer B.SilkS)
+  (gr_text "Cherry MX version\nRev. 1.0.1" (at 148.336 109.601) (layer B.SilkS)
     (effects (font (size 1 1) (thickness 0.2)) (justify left mirror))
   )

Commit message: development version
Other:
- board text added: "Cherry MX version Rev. develop"
- board text removed: "Cherry MX version Rev. 1.0.1"
Changed lines of the file:
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@@
     (effects (font (size 1 1.4) (thickness 0.2)) (justify mirror))
   )
-  (gr_text "Cherry MX version\nRev. 1.0.1" (at 148.336 109.601) (layer B.SilkS)
+  (gr_text "Cherry MX version\nRev. develop" (at 148.336 109.601) (layer B.SilkS)
     (effects (font (size 1 1) (thickness 0.2)) (justify left mirror))
   )

Commit message: merge `hanya/let-s-Split-v2`
Parts:
- added J4: 3PIN, local:CON3_SMD_BOTH, F.Cu at (40.0, 73.0)
- added J5: 3PIN, local:CON3_SMD_BOTH, F.Cu at (146.0, 73.0)
- added M1: FIDUCIAL, local:Fiducial_Mark, F.Cu at (40.0, 50.4)
- added M2: FIDUCIAL, local:Fiducial_Mark, F.Cu at (145.8, 108.3)
- added M3: FIDUCIAL, local:Fiducial_Mark, B.Cu at (145.8, 108.3)
- added M4: FIDUCIAL, local:Fiducial_Mark, B.Cu at (40.0, 50.4)
- added RSW1: SW_PUSH, local:TACTILE_COMPATIBLE, F.Cu at (78.8, 35.9)
- D1, D10, D11, D12, D13, D14, D15, D16, D17, D18, D19, D2, D20, D21, D22, D23, D24, D3, D4, D5, D6, D7, D8, D9: footprint Diodes_ThroughHole:Diode_DO-41_SOD81_Horizontal_RM10 -> local:Diode_TH_SOD123
- J1: footprint prettylib:jumper -> local:SMD_JUMPER_2
- J3: footprint prettylib:jumper -> local:SMD_JUMPER_2; moved to B.Cu
- R1, R2: value R -> 4K7; footprint footprint:RESISTOR -> local:RESISTOR
- SW1, SW10, SW11, SW12, SW13, SW14, SW15, SW16, SW17, SW18, SW19, SW2, SW21, SW22, SW23, SW3, SW4, SW5, SW6, SW7, SW8, SW9: footprint flipalps:MXALPS_FLIP -> local:MXALPS_FLIP_HOLES
- SW20, SW24: renamed from ?; footprint flipalps:MXALPS_FLIP -> local:MXALPS_FLIP_HOLES
- U1: value (none) -> ProMicro; footprint footprint:TEENSY_2.0 -> local:ProMicro; moved to F.Cu
- moved D5 11.7 mm to (76.9, 56.3), turned to 0 degrees
- moved D1 10.2 mm to (40.8, 56.4), turned to 0 degrees
- moved D2 6.55 mm to (43.5, 75.4), turned to 0 degrees
- moved J1 3.10 mm to (136.4, 50.3), turned to 0 degrees
- moved D22 2.60 mm to (133.0, 75.3)
- moved D17 1.50 mm to (115.2, 56.3)
- moved R1 1.50 mm to (94.9, 56.3)
- moved R2 1.50 mm to (107.5, 56.3)
- moved D21 1.10 mm to (137.0, 56.2)
- moved J3 1.03 mm to (126.9, 50.3), turned to 0 degrees
- moved D18 1.00 mm to (131.3, 72.5)
- moved W2 0.86 mm to (131.7, 47.5)
- turned W1 to 180 degrees
Connections:
- R1 pad 2: Net-(R1-Pad2) -> I2C_SDA
- U1 pad 10: col3 -> row1
- U1 pad 11: col4 -> row2
- U1 pad 12: col5 -> row3
- U1 pad 18: row3 -> col0
- U1 pad 19: row2 -> (no net)
- U1 pad 2: GND -> (no net)
- U1 pad 20: row1 -> (no net)
- U1 pad 21: row0 -> VCC
- U1 pad 23: Net-(U1-Pad23) -> GND
- U1 pad 24: data -> (no net)
- U1 pad 3: Net-(U1-Pad3) -> GND
- U1 pad 4: VCC -> GND
- U1 pad 5: Net-(U1-Pad5) -> I2C_SDA
- U1 pad 6: Net-(U1-Pad6) -> data
- U1 pad 7: col0 -> (no net)
- U1 pad 8: col1 -> (no net)
- U1 pad 9: col2 -> row0
- W1 pad 2: Net-(R1-Pad2) -> I2C_SDA
Routing:
- net GND: track 15.8 -> 743.8 mm, vias 0 -> 54
- net VCC: track 27.2 -> 187.1 mm, vias 0 -> 8
- net Net-(R1-Pad2): track 77.0 -> 0.00 mm, vias 1 -> 0
- net I2C_SDA: track 0.00 -> 73.0 mm, vias 0 -> 1
- net Net-(J4-Pad2): track 0.00 -> 56.5 mm, vias 0 -> 2
- net row0: track 96.8 -> 150.3 mm, vias 0 -> 1
- net row1: track 108.7 -> 153.0 mm, vias 0 -> 1
- net row3: track 142.8 -> 183.6 mm
- net row2: track 121.1 -> 156.7 mm
- net xtradata: track 25.8 -> 55.4 mm, vias 0 -> 2
- net data: track 117.4 -> 97.4 mm, vias 0 -> 1
- net Net-(D5-Pad2): track 22.9 -> 36.8 mm, vias 0 -> 1
- net col5: track 139.6 -> 150.8 mm, vias 0 -> 1
- net Net-(D24-Pad2): track 33.6 -> 44.0 mm
- net Net-(D21-Pad2): track 16.4 -> 24.1 mm
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- added copper zone on B.Cu, net GND
- removed copper zone on B.Cu, net VCC
Other:
- board size 112 x 79 mm -> 111.8 x 79 mm
- net class Default: clearance 0.2 -> 0
- rule trace_clearance: 0.2 -> 0
- board text added: "Connect them if jack is on this side."
- board text added: "DO/Din"
- board text added: "Designed by Wootpatoot"
- board text added: "Din"
- board text added: "Din/DO"
- board text added: "I2C pull-ups"
- board text added: "J1"
- board text added: "J3"
- board text added: "J4"
- board text added: "J5"
- board text added: "LED Strip"
- board text added: "Pro Micro"
- board text added: "Reset"
- board text added: "U1"
- board text removed: "By Wootpatoot"

Commit message: bump version to 1.1.0
Other:
- board text added: "Cherry MX version Rev. 1.1.0"
- board text removed: "Cherry MX version Rev. develop"
Changed lines of the file:
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@@
       (net 29 GND))
   )
-  (gr_text "Cherry MX version\nRev. develop" (at 38.735 109.347) (layer B.SilkS)
+  (gr_text "Cherry MX version\nRev. 1.1.0" (at 38.735 109.347) (layer B.SilkS)
     (effects (font (size 1 1) (thickness 0.2)) (justify right mirror))
   )

Commit message: Use local holes and JUMPER_SMD_2DUB
Parts:
- U2, U3, U4: footprint prettylib:HOLE -> local:HOLE
- U5: footprint prettylib:HOLE -> local:HOLE_2
- W1: footprint prettylib:JUMPER_SMD_2DUB -> local:JUMPER_SMD_2DUB
