File: lets_split.sch (KiCad schematic (older format))
At the start: 67 parts, among them J1 3PIN, J2 6PIN, J3 3PIN, J4 3PIN, J5 3PIN, M1 FIDUCIAL, M2 FIDUCIAL, M3 FIDUCIAL, M4 FIDUCIAL, SW1 SW_PUSH, SW10 SW_PUSH, SW11 SW_PUSH, SW12 SW_PUSH, SW13 SW_PUSH, SW14 SW_PUSH, SW15 SW_PUSH, SW16 SW_PUSH, SW17 SW_PUSH, SW18 SW_PUSH, SW19 SW_PUSH, SW2 SW_PUSH, SW20 SW_PUSH, SW21 SW_PUSH, SW22 SW_PUSH, SW23 SW_PUSH, SW24 SW_PUSH, SW3 SW_PUSH, SW4 SW_PUSH, SW5 SW_PUSH, SW6 SW_PUSH, SW7 SW_PUSH, SW8 SW_PUSH, SW9 SW_PUSH, U1 ProMicro, U2 HOLE, U3 HOLE, U4 HOLE, U5 HOLE

Commit message: Add universal switch; fix prettylib
Parts:
- SW1, SW10, SW11, SW12, SW13, SW14, SW15, SW16, SW17, SW18, SW19, SW2, SW20, SW21, SW22, SW23, SW24, SW3, SW4, SW5, SW6, SW7, SW8, SW9: footprint local:MXALPS_FLIP_HOLES -> local:MX-ALPs-PG1350-FLIP
- U2, U3, U4, U5: footprint prettylib:HOLE -> local:HOLE
- W1: footprint prettylib:JUMPER_SMD_2DUB -> local:JUMPER_SMD_2DUB
Changed lines of the file:
@@
 F 0 "SW1" H 5600 3310 50  0000 C CNN
 F 1 "SW_PUSH" H 5450 3120 50  0000 C CNN
-F 2 "local:MXALPS_FLIP_HOLES" H 5450 3200 50  0001 C CNN
+F 2 "local:MX-ALPs-PG1350-FLIP" H 5450 3200 50  0001 C CNN
 F 3 "" H 5450 3200 50  0000 C CNN
 	1    5450 3200
@@
 F 0 "SW5" H 6350 3310 50  0000 C CNN
 F 1 "SW_PUSH" H 6200 3120 50  0000 C CNN
-F 2 "local:MXALPS_FLIP_HOLES" H 6200 3200 50  0001 C CNN
+F 2 "local:MX-ALPs-PG1350-FLIP" H 6200 3200 50  0001 C CNN
 F 3 "" H 6200 3200 50  0000 C CNN
 	1    6200 3200
@@
 F 0 "SW9" H 7050 3310 50  0000 C CNN
 F 1 "SW_PUSH" H 6900 3120 50  0000 C CNN
-F 2 "local:MXALPS_FLIP_HOLES" H 6900 3200 50  0001 C CNN
+F 2 "local:MX-ALPs-PG1350-FLIP" H 6900 3200 50  0001 C CNN
 F 3 "" H 6900 3200 50  0000 C CNN
 	1    6900 3200
@@
 F 0 "SW13" H 7800 3310 50  0000 C CNN
 F 1 "SW_PUSH" H 7650 3120 50  0000 C CNN
-F 2 "local:MXALPS_FLIP_HOLES" H 7650 3200 50  0001 C CNN
+F 2 "local:MX-ALPs-PG1350-FLIP" H 7650 3200 50  0001 C CNN
 F 3 "" H 7650 3200 50  0000 C CNN
 	1    7650 3200
@@
 F 0 "SW17" H 8550 3310 50  0000 C CNN
 F 1 "SW_PUSH" H 8400 3120 50  0000 C CNN
-F 2 "local:MXALPS_FLIP_HOLES" H 8400 3200 50  0001 C CNN
+F 2 "local:MX-ALPs-PG1350-FLIP" H 8400 3200 50  0001 C CNN
 F 3 "" H 8400 3200 50  0000 C CNN
 	1    8400 3200
@@
 F 0 "SW21" H 9300 3310 50  0000 C CNN
 F 1 "SW_PUSH" H 9150 3120 50  0000 C CNN
-F 2 "local:MXALPS_FLIP_HOLES" H 9150 3200 50  0001 C CNN
+F 2 "local:MX-ALPs-PG1350-FLIP" H 9150 3200 50  0001 C CNN
 F 3 "" H 9150 3200 50  0000 C CNN
 	1    9150 3200
@@
 F 0 "SW2" H 5600 3810 50  0000 C CNN
 F 1 "SW_PUSH" H 5450 3620 50  0000 C CNN
-F 2 "local:MXALPS_FLIP_HOLES" H 5450 3700 50  0001 C CNN
+F 2 "local:MX-ALPs-PG1350-FLIP" H 5450 3700 50  0001 C CNN
 F 3 "" H 5450 3700 50  0000 C CNN
 	1    5450 3700
@@
 F 0 "SW6" H 6350 3810 50  0000 C CNN
 F 1 "SW_PUSH" H 6200 3620 50  0000 C CNN
-F 2 "local:MXALPS_FLIP_HOLES" H 6200 3700 50  0001 C CNN
+F 2 "local:MX-ALPs-PG1350-FLIP" H 6200 3700 50  0001 C CNN
 F 3 "" H 6200 3700 50  0000 C CNN
 	1    6200 3700
@@
 F 0 "SW10" H 7050 3810 50  0000 C CNN
 F 1 "SW_PUSH" H 6900 3620 50  0000 C CNN
-F 2 "local:MXALPS_FLIP_HOLES" H 6900 3700 50  0001 C CNN
+F 2 "local:MX-ALPs-PG1350-FLIP" H 6900 3700 50  0001 C CNN
 F 3 "" H 6900 3700 50  0000 C CNN
 	1    6900 3700
@@
 F 0 "SW14" H 7800 3810 50  0000 C CNN
 F 1 "SW_PUSH" H 7650 3620 50  0000 C CNN
-F 2 "local:MXALPS_FLIP_HOLES" H 7650 3700 50  0001 C CNN
+F 2 "local:MX-ALPs-PG1350-FLIP" H 7650 3700 50  0001 C CNN
 F 3 "" H 7650 3700 50  0000 C CNN
 	1    7650 3700
@@
 F 0 "SW18" H 8550 3810 50  0000 C CNN
 F 1 "SW_PUSH" H 8400 3620 50  0000 C CNN
-F 2 "local:MXALPS_FLIP_HOLES" H 8400 3700 50  0001 C CNN
+F 2 "local:MX-ALPs-PG1350-FLIP" H 8400 3700 50  0001 C CNN
 F 3 "" H 8400 3700 50  0000 C CNN
 	1    8400 3700
@@
 F 0 "SW22" H 9300 3810 50  0000 C CNN
 F 1 "SW_PUSH" H 9150 3620 50  0000 C CNN
-F 2 "local:MXALPS_FLIP_HOLES" H 9150 3700 50  0001 C CNN
+F 2 "local:MX-ALPs-PG1350-FLIP" H 9150 3700 50  0001 C CNN
 F 3 "" H 9150 3700 50  0000 C CNN
 	1    9150 3700
@@
 F 0 "SW3" H 5600 4310 50  0000 C CNN
 F 1 "SW_PUSH" H 5450 4120 50  0000 C CNN
-F 2 "local:MXALPS_FLIP_HOLES" H 5450 4200 50  0001 C CNN
+F 2 "local:MX-ALPs-PG1350-FLIP" H 5450 4200 50  0001 C CNN
 F 3 "" H 5450 4200 50  0000 C CNN
 	1    5450 4200
@@
 F 0 "SW7" H 6350 4310 50  0000 C CNN
 F 1 "SW_PUSH" H 6200 4120 50  0000 C CNN
-F 2 "local:MXALPS_FLIP_HOLES" H 6200 4200 50  0001 C CNN
+F 2 "local:MX-ALPs-PG1350-FLIP" H 6200 4200 50  0001 C CNN
 F 3 "" H 6200 4200 50  0000 C CNN
 	1    6200 4200
@@
 F 0 "SW11" H 7050 4310 50  0000 C CNN
 F 1 "SW_PUSH" H 6900 4120 50  0000 C CNN
-F 2 "local:MXALPS_FLIP_HOLES" H 6900 4200 50  0001 C CNN
+F 2 "local:MX-ALPs-PG1350-FLIP" H 6900 4200 50  0001 C CNN
 F 3 "" H 6900 4200 50  0000 C CNN
 	1    6900 4200
@@
 F 0 "SW15" H 7800 4310 50  0000 C CNN
 F 1 "SW_PUSH" H 7650 4120 50  0000 C CNN
-F 2 "local:MXALPS_FLIP_HOLES" H 7650 4200 50  0001 C CNN
+F 2 "local:MX-ALPs-PG1350-FLIP" H 7650 4200 50  0001 C CNN
 F 3 "" H 7650 4200 50  0000 C CNN
 	1    7650 4200
@@
 F 0 "SW19" H 8550 4310 50  0000 C CNN
 F 1 "SW_PUSH" H 8400 4120 50  0000 C CNN
-F 2 "local:MXALPS_FLIP_HOLES" H 8400 4200 50  0001 C CNN
+F 2 "local:MX-ALPs-PG1350-FLIP" H 8400 4200 50  0001 C CNN
 F 3 "" H 8400 4200 50  0000 C CNN
 	1    8400 4200
@@
 F 0 "SW23" H 9300 4310 50  0000 C CNN
 F 1 "SW_PUSH" H 9150 4120 50  0000 C CNN
-F 2 "local:MXALPS_FLIP_HOLES" H 9150 4200 50  0001 C CNN
+F 2 "local:MX-ALPs-PG1350-FLIP" H 9150 4200 50  0001 C CNN
 F 3 "" H 9150 4200 50  0000 C CNN
 	1    9150 4200
@@
 F 0 "SW4" H 5600 4810 50  0000 C CNN
 F 1 "SW_PUSH" H 5450 4620 50  0000 C CNN
-F 2 "local:MXALPS_FLIP_HOLES" H 5450 4700 50  0001 C CNN
+F 2 "local:MX-ALPs-PG1350-FLIP" H 5450 4700 50  0001 C CNN
 F 3 "" H 5450 4700 50  0000 C CNN
 	1    5450 4700
@@
 F 0 "SW8" H 6350 4810 50  0000 C CNN
 F 1 "SW_PUSH" H 6200 4620 50  0000 C CNN
-F 2 "local:MXALPS_FLIP_HOLES" H 6200 4700 50  0001 C CNN
+F 2 "local:MX-ALPs-PG1350-FLIP" H 6200 4700 50  0001 C CNN
 F 3 "" H 6200 4700 50  0000 C CNN
 	1    6200 4700
@@
 F 0 "SW12" H 7050 4810 50  0000 C CNN
 F 1 "SW_PUSH" H 6900 4620 50  0000 C CNN
-F 2 "local:MXALPS_FLIP_HOLES" H 6900 4700 50  0001 C CNN
+F 2 "local:MX-ALPs-PG1350-FLIP" H 6900 4700 50  0001 C CNN
 F 3 "" H 6900 4700 50  0000 C CNN
 	1    6900 4700
@@
 F 0 "SW16" H 7800 4810 50  0000 C CNN
 F 1 "SW_PUSH" H 7650 4620 50  0000 C CNN
-F 2 "local:MXALPS_FLIP_HOLES" H 7650 4700 50  0001 C CNN
+F 2 "local:MX-ALPs-PG1350-FLIP" H 7650 4700 50  0001 C CNN
 F 3 "" H 7650 4700 50  0000 C CNN
 	1    7650 4700
@@
 F 0 "SW20" H 8550 4810 50  0000 C CNN
 F 1 "SW_PUSH" H 8400 4620 50  0000 C CNN
-F 2 "local:MXALPS_FLIP_HOLES" H 8400 4700 50  0001 C CNN
+F 2 "local:MX-ALPs-PG1350-FLIP" H 8400 4700 50  0001 C CNN
 F 3 "" H 8400 4700 50  0000 C CNN
 	1    8400 4700
@@
 F 0 "SW24" H 9300 4810 50  0000 C CNN
 F 1 "SW_PUSH" H 9150 4620 50  0000 C CNN
-F 2 "local:MXALPS_FLIP_HOLES" H 9150 4700 50  0001 C CNN
+F 2 "local:MX-ALPs-PG1350-FLIP" H 9150 4700 50  0001 C CNN
 F 3 "" H 9150 4700 50  0000 C CNN
 	1    9150 4700
@@
 F 0 "W1" H 7350 1210 50  0000 C CNN
 F 1 "TEST" H 7350 1080 50  0000 C CNN
-F 2 "prettylib:JUMPER_SMD_2DUB" H 7350 1150 50  0001 C CNN
+F 2 "local:JUMPER_SMD_2DUB" H 7350 1150 50  0001 C CNN
 F 3 "" H 7350 1150 50  0000 C CNN
 	1    7350 1150
@@
 F 0 "U2" H 5200 7250 60  0000 C CNN
 F 1 "HOLE" H 5200 7050 60  0000 C CNN
-F 2 "prettylib:HOLE" H 5200 7050 60  0001 C CNN
+F 2 "local:HOLE" H 5200 7050 60  0001 C CNN
 F 3 "" H 5200 7050 60  0000 C CNN
 	1    5200 7050
@@
 F 0 "U3" H 5600 7250 60  0000 C CNN
 F 1 "HOLE" H 5600 7050 60  0000 C CNN
-F 2 "prettylib:HOLE" H 5600 7050 60  0001 C CNN
+F 2 "local:HOLE" H 5600 7050 60  0001 C CNN
 F 3 "" H 5600 7050 60  0000 C CNN
 	1    5600 7050
@@
 F 0 "U4" H 6000 7250 60  0000 C CNN
 F 1 "HOLE" H 6000 7050 60  0000 C CNN
-F 2 "prettylib:HOLE" H 6000 7050 60  0001 C CNN
+F 2 "local:HOLE" H 6000 7050 60  0001 C CNN
 F 3 "" H 6000 7050 60  0000 C CNN
 	1    6000 7050
@@
 F 0 "U5" H 6400 7250 60  0000 C CNN
 F 1 "HOLE" H 6400 7050 60  0000 C CNN
-F 2 "prettylib:HOLE" H 6400 7050 60  0001 C CNN
+F 2 "local:HOLE" H 6400 7050 60  0001 C CNN
 F 3 "" H 6400 7050 60  0000 C CNN
 	1    6400 7050
